File: CAN_BDC_Driver/BDC_CAN/BDC_CAN.kicad_pcb (KiCad board)
At the start: 2 copper layers, 87 x 91.6 mm, 56 parts, among them J1 VCC_IN, J2 Motor1_Out, J3 Motor2_Out, J4 CAN, J5 USB_C_Receptacle_USB2.0_16P, J6 Conn_01x05_Pin, Q1 PMOS, Q2 NMOS, Q3 PMOS, Q4 NMOS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

Commit message: Placement Changed
Parts:
- moved C11 61.0 mm to (85.5, 35.8)
- moved C15 61.0 mm to (143.1, 73.0)
- moved C5 61.0 mm to (109.5, 51.1)
- moved J4 61.0 mm to (81.5, 25.9)
- moved Q2 61.0 mm to (104.1, 34.0)
- moved Q5 61.0 mm to (132.0, 80.5)
- moved R4 61.0 mm to (140.8, 51.5)
- moved C1 61.0 mm to (114.9, 56.8)
- moved C10 61.0 mm to (104.1, 63.0)
- moved C3 61.0 mm to (107.7, 51.1)
- moved C7 61.0 mm to (113.1, 51.1)
- moved C9 61.0 mm to (98.7, 73.2)
- moved D2 61.0 mm to (126.7, 71.8)
- moved D5 61.0 mm to (121.9, 71.6)
- moved G*** 61.0 mm to (88.3, 57.8)
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
Commit message: New Design
Parts:
- removed G*** (x2): LOGO, LOGO
- removed SW2: SW_DIP_x06, Button_Switch_SMD:SW_DIP_SPSTx06_Slide_6.7x16.8mm_W6.73mm_P2.54mm_LowProfile_JPin
- added J7: Conn_01x05_Pin, Connector_JST:JST_PH_S5B-PH-K_1x05_P2.00mm_Horizontal, F.Cu at (152.3, 42.3)
- C1, C10, C2, C3, C5, C6, C7, C8, C9, U2, Y1: moved to F.Cu
- U4: moved to B.Cu
- moved J4 145.3 mm to (224.5, 52.0)
- moved U5 144.5 mm to (217.6, 114.7), turned to 0 degrees
- moved J3 126.5 mm to (54.6, 165.3)
- moved J2 105.7 mm to (40.4, 53.1)
- moved SW1 98.2 mm to (168.5, 60.4), turned to 0 degrees
- moved Q4 91.5 mm to (49.5, 82.2)
- moved Q7 89.5 mm to (25.0, 112.3)
- moved Q1 87.6 mm to (19.5, 82.2)
- moved R7 86.0 mm to (162.3, 104.8), turned to 0 degrees
- moved C15 85.4 mm to (113.5, 153.0)
- moved R6 85.3 mm to (173.3, 36.5), turned to 0 degrees
- moved Q5 84.9 mm to (53.0, 111.8)
- moved C17 84.3 mm to (125.3, 153.0)
- moved Q2 83.9 mm to (35.5, 82.2)
- moved C11 83.8 mm to (169.2, 39.0), turned to 0 degrees
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Connections:
- J2 pad 1: /Driver+FETS/MB -> /Driver+FETS/MA
- J2 pad 2: /Driver+FETS/MA -> /Driver+FETS/MB
- J3 pad 1: /Driver+FETS1/MB -> /Driver+FETS1/MA
- J3 pad 2: /Driver+FETS1/MA -> /Driver+FETS1/MB
- U1 pad 29: /mC/DIP6 -> unconnected-(U1-PA8-Pad29)
- U1 pad 30: /mC/DIP5 -> unconnected-(U1-PA9-Pad30)
- U1 pad 31: /mC/DIP4 -> unconnected-(U1-PA10-Pad31)
- U1 pad 38: /mC/DIP3 -> unconnected-(U1-PA15-Pad38)
- U1 pad 39: /mC/DIP2 -> /mC/SDA
- U1 pad 40: /mC/DIP1 -> /mC/SCL
Routing:
- net /Driver+FETS/5V: track 135.3 -> 0.00 mm, vias 3 -> 0
- net /Driver+FETS/VCC: track 128.8 -> 0.00 mm, vias 1 -> 0
- net GND: track 100.5 -> 0.00 mm, vias 17 -> 0
- net /Driver+FETS/MA: track 79.8 -> 0.00 mm
- net /Driver+FETS1/MB: track 76.2 -> 0.00 mm
- net +3.3V: track 50.4 -> 0.00 mm, vias 2 -> 0
- net /Driver+FETS1/MA: track 45.8 -> 0.00 mm
- net /mC/CAN_H: track 45.0 -> 0.00 mm, vias 2 -> 0
- net /mC/CAN_L: track 43.2 -> 0.00 mm, vias 2 -> 0
- net /mC/UART_RX: track 41.5 -> 0.00 mm, vias 2 -> 0
- net /Driver+FETS/MB: track 41.2 -> 0.00 mm
- net /mC/UART_TX: track 40.2 -> 0.00 mm, vias 2 -> 0
- net USB_D-: track 34.9 -> 0.00 mm, vias 2 -> 0
- net Net-(C4-Pad2): track 34.5 -> 0.00 mm, vias 2 -> 0
- net USB_D+: track 28.1 -> 0.00 mm, vias 2 -> 0
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- added copper zone on F.Cu, net /Driver+FETS/MA
- added copper zone on F.Cu, net /Driver+FETS/MB
- removed copper zone on B.Cu, net GND
Other:
- board outline removed
- board text removed: "Anirudha Duttagupta"
