File: CAN_BDC_Driver/BDC_CAN/BDC_CAN.kicad_sch (KiCad schematic)
At the start: 4 parts, among them J1 VCC_IN, J2 Motor1_Out, J3 Motor2_Out, J4 CAN

Commit message: New Design
Connections:
- net Driver+FETS/MA: now also J2.1 (Pin_1); no longer J2.2 (Pin_2)
- net Driver+FETS/MB: now also J2.2 (Pin_2); no longer J2.1 (Pin_1)
- net Driver+FETS1/MA: now also J3.1 (Pin_1); no longer J3.2 (Pin_2)
- net Driver+FETS1/MB: now also J3.2 (Pin_2); no longer J3.1 (Pin_1)
Other:
- moved on the sheet: J2, J3
Changed lines of the file:
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@@
 	(symbol
 		(lib_id "Connector:Conn_01x02_Pin")
-		(at 207.01 86.36 180)
-		(unit 1)
-		(exclude_from_sim no)
-		(in_bom yes)
-		(on_board yes)
-		(dnp no)
-		(fields_autoplaced yes)
+		(at 207.01 83.82 0)
+		(mirror y)
+		(unit 1)
+		(exclude_from_sim no)
+		(in_bom yes)
+		(on_board yes)
+		(dnp no)
 		(property "Reference" "J2"
-			(at 208.28 83.8199 0)
+			(at 208.28 86.3601 0)
 			(effects
 				(font
@@
 		)
 		(property "Value" "Motor1_Out"
-			(at 208.28 86.3599 0)
+			(at 208.28 83.8201 0)
 			(effects
 				(font
@@
 		)
 		(property "Footprint" "Connector_AMASS:AMASS_XT60PW-M_1x02_P7.20mm_Horizontal"
-			(at 207.01 86.36 0)
-			(effects
-				(font
-					(size 1.27 1.27)
-				)
-				(hide yes)
-			)
-		)
-		(property "Datasheet" "~"
-			(at 207.01 86.36 0)
-			(effects
-				(font
-					(size 1.27 1.27)
-				)
-				(hide yes)
-			)
-		)
-		(property "Description" "Generic connector, single row, 01x02, script generated"
-			(at 207.01 86.36 0)
+			(at 207.01 83.82 0)
+			(effects
+				(font
+					(size 1.27 1.27)
+				)
+				(hide yes)
+			)
+		)
+		(property "Datasheet" "~"
+			(at 207.01 83.82 0)
+			(effects
+				(font
+					(size 1.27 1.27)
+				)
+				(hide yes)
+			)
+		)
+		(property "Description" "Generic connector, single row, 01x02, script generated"
+			(at 207.01 83.82 0)
 			(effects
 				(font
@@
 	(symbol
 		(lib_id "Connector:Conn_01x02_Pin")
-		(at 209.55 125.73 180)
-		(unit 1)
-		(exclude_from_sim no)
-		(in_bom yes)
-		(on_board yes)
-		(dnp no)
-		(fields_autoplaced yes)
+		(at 209.55 123.19 0)
+		(mirror y)
+		(unit 1)
+		(exclude_from_sim no)
+		(in_bom yes)
+		(on_board yes)
+		(dnp no)
 		(property "Reference" "J3"
-			(at 210.82 123.1899 0)
+			(at 210.82 125.7301 0)
 			(effects
 				(font
@@
 		)
 		(property "Value" "Motor2_Out"
-			(at 210.82 125.7299 0)
+			(at 210.82 123.1901 0)
 			(effects
 				(font
@@
 		)
 		(property "Footprint" "Connector_AMASS:AMASS_XT60PW-M_1x02_P7.20mm_Horizontal"
-			(at 209.55 125.73 0)
-			(effects
-				(font
-					(size 1.27 1.27)
-				)
-				(hide yes)
-			)
-		)
-		(property "Datasheet" "~"
-			(at 209.55 125.73 0)
-			(effects
-				(font
-					(size 1.27 1.27)
-				)
-				(hide yes)
-			)
-		)
-		(property "Description" "Generic connector, single row, 01x02, script generated"
-			(at 209.55 125.73 0)
-			(effects
-				(font
+			(at 209.55 123.19 0)
+			(effects
+				(font
+					(size 1.27 1.27)
+				)
+				(hide yes)
+			)
+		)
+		(property "Datasheet" "~"
+			(at 209.55 123.19 0)
+			(effects
+				(font
+					(size 1.27 1.27)
+				)
+				(hide yes)
+			)
+		)
+		(property "Description" "Generic connector, single row, 01x02, script generated"
+			(at 209.55 123.19 0)
+			(effects
+				(font
